File: docs/schematic/schematic.kicad_pcb (KiCad board)
At the start: 2 copper layers, 83.8 x 61 mm, 9 parts, among them J1 AudioJack2, SW1 SW_Push, SW2 SW_Push, SW3 SW_Push, SW4 SW_Push, U1 Pico

Commit message: Update Schematic to as built
We deviated from the original schematic as it was simpler to construct/ source in the way we built  it.
Parts:
- added R2: 250, Resistor_THT:R_Axial_DIN0309_L9.0mm_D3.2mm_P15.24mm_Horizontal, F.Cu at (35.6, 25.4)
- J1: value AudioJack2 -> AudioJack3; footprint Connector_Wire:SolderWire-0.15sqmm_1x02_P4mm_D0.5mm_OD1.5mm -> Connector_Audio:Jack_6.35mm_Neutrik_NJ3FD-V_Vertical
- moved R1 15.9 mm to (40.6, 25.4), turned to -90 degrees
- moved J1 6.10 mm to (22.9, 19.7), turned to 0 degrees
- moved SW1 0.16 mm to (17.8, 45.7)
Connections:
- net Net-(RV1-Pad3) renamed VCC
- J1 pad T: Net-(U1-Pad3) -> Net-(J1-PadT)
- R1 pad 1: Net-(J1-PadS) -> Net-(J1-PadR)
- SW3 pad 1: Net-(SW1-Pad1) -> Net-(SW3-Pad1)
- SW4 pad 1: Net-(SW1-Pad1) -> Net-(SW3-Pad1)
- U1 pad 13: unconnected-(U1-Pad13) -> Net-(SW1-Pad1)
- U1 pad 18: Net-(SW1-Pad1) -> Net-(SW3-Pad1)
- U1 pad 3: Net-(U1-Pad3) -> Net-(J1-PadS)
- U1 pad 5: unconnected-(U1-Pad5) -> Net-(R2-Pad2)
Routing:
- net Net-(SW3-Pad1): track 0.00 -> 42.7 mm
- net Net-(J1-PadS): track 5.53 -> 37.3 mm
- net Net-(U1-Pad3): track 30.4 -> 0.00 mm
- net Net-(R2-Pad2): track 0.00 -> 19.6 mm
- net Net-(SW1-Pad1): track 57.9 -> 41.9 mm
- net Net-(J1-PadT): track 0.00 -> 15.1 mm
- net Net-(J1-PadR): track 0.00 -> 14.1 mm
- net Net-(R1-Pad2): track 11.2 -> 17.1 mm
- net Net-(SW1-Pad2): track 33.0 -> 32.2 mm
